Commit message: fix: tune up torque

File: www/static/robot.urdf (robot description, URDF)
Before this commit: robot onshape_to_robot_6a409ed450e730.23812679, 46 links, 45 joints
Links:
- link body: mass 0.161638 -> 0.10137; geometry visual mesh filename=package://assets/battery_cap_thin.stl; visual mesh filename=package://assets/body.stl
